Commit message: updating robot colors, position and stop condition

File: Go-chase-it/catkin_ws/src/my_robot/urdf/my_robot.xacro (robot description, xacro)
@@ -1,15 +1,6 @@
 <?xml version='1.0'?>
 <robot name="my_robot" xmlns:xacro="http://www.ros.org/wiki/xacro">
-  <material name="orange">
-    <color rgba="${255/255} ${108/255} ${10/255} 1.0"/>
-  </material>
-  <material name="blue">
-    <color rgba="0 0 0.8 1"/>
-  </material>
-  <material name="white">
-    <color rgba="1 1 1 1"/>
-  </material>
+  <link name="robot_footprint"></link>
   <xacro:include filename="$(find my_robot)/urdf/my_robot.gazebo" />
-  <link name="robot_footprint"></link>
   <joint name="robot_footprint_joint" type="fixed">
     <origin xyz="0 0 0" rpy="0 0 0" />
@@ -33,5 +24,4 @@
         <box size=".4 .2 .1"/>
       </geometry>
-      <material name="orange"/>
     </collision>
     <visual name='chassis_visual'>
@@ -40,5 +30,4 @@
         <box size=".4 .2 .1"/>
       </geometry>
-      <material name="orange"/>
     </visual>
     <collision name='back_caster_collision'>
@@ -67,4 +56,7 @@
     </visual>
   </link>
+  <gazebo reference='chassis'>
+	<material>Gazebo/Red</material>
+  </gazebo>
   <link name='left_wheel'>
     <pose>0 0 0.1 0 0 0</pose>
@@ -83,5 +75,4 @@
         <cylinder radius="0.1" length="0.05"/>
       </geometry>
-      <material name="white"/>
     </collision>
     <visual name='left_wheel_visual'>
@@ -90,7 +81,9 @@
         <cylinder radius="0.1" length="0.05"/>
       </geometry>
-      <material name="white"/>
-    </visual>
-  </link>
+    </visual>
+  </link>
+  <gazebo reference='left_wheel'>
+	<material>Gazebo/Green</material>
+  </gazebo>
   <joint type="continuous" name="left_wheel_hinge">
     <origin xyz="0 0.15 0" rpy="0 0 0"/>
@@ -117,5 +110,4 @@
         <cylinder radius="0.1" length="0.05"/>
       </geometry>
-      <material name="white"/>
     </collision>
     <visual name='right_wheel_visual'>
@@ -124,7 +116,9 @@
         <cylinder radius="0.1" length="0.05"/>
       </geometry>
-      <material name="white"/>
-    </visual>
-  </link>
+    </visual>
+  </link>
+  <gazebo reference='right_wheel'>
+	<material>Gazebo/Green</material>
+  </gazebo>
   <joint type="continuous" name="right_wheel_hinge">
     <origin xyz="0 -0.15 0" rpy="0 0 0"/>
@@ -149,16 +143,17 @@
       <origin xyz="0 0 0" rpy=" 0 0 0"/>
       <geometry>
-        <box size="0.05 0.05 0.05"/>
-      </geometry>
-      <material name="blue"/>
+        <box size="0.01 0.05 0.05"/>
+      </geometry>
     </collision>
     <visual name='camera_visual'>
       <origin xyz="0 0 0" rpy=" 0 0 0"/>
       <geometry>
-        <box size="0.05 0.05 0.05"/>
-      </geometry>
-      <material name="blue"/>
-    </visual>
-  </link>
+        <box size="0.01 0.05 0.05"/>
+      </geometry>
+    </visual>
+  </link>
+  <gazebo reference='camera'>
+	<material>Gazebo/Black</material>
+  </gazebo>
   <joint type="fixed" name="camera_joint">
     <origin xyz="0.2 0 0" rpy="0 0 0"/>
@@ -201,3 +196,7 @@
     <dynamics damping="1.0" friction="1.0"/>
   </joint>
+<gazebo>
+  <plugin name="gazebo_ros_control" filename="libgazebo_ros_control.so">
+  </plugin>
+</gazebo>
 </robot>
