Commit message: Update of my_robot xacro file: correct the configuration of sensor RGB-D camera

File: Map-my-world/catkin_ws/src/my_robot/urdf/my_robot.xacro (robot description, xacro)
@@ -1,6 +1,6 @@
 <?xml version='1.0'?>
 <robot name="my_robot" xmlns:xacro="http://www.ros.org/wiki/xacro">
+<xacro:include filename="$(find my_robot)/urdf/my_robot.gazebo" />
   <link name="robot_footprint"></link>
-  <xacro:include filename="$(find my_robot)/urdf/my_robot.gazebo" />
   <joint name="robot_footprint_joint" type="fixed">
     <origin xyz="0 0 0" rpy="0 0 0" />
@@ -164,4 +164,32 @@
     <dynamics damping="1.0" friction="1.0"/>
   </joint>
+<link name="camera_rgbd">
+     <visual>
+      <origin xyz="0 0 0" rpy="0 0 0"/>
+       <geometry>
+        <box size=".05 .05 .05"/>
+      </geometry>
+    </visual>
+    <inertial>
+      <mass value="0.1"/>
+      <origin xyz="0 0 0" rpy=" 0 0 0"/>
+      <inertia
+          ixx="0.000001" ixy="0" ixz="0"
+          iyy="0.000001" iyz="0"
+          izz="0.000001"
+      />
+    </inertial>
+    <collision>
+      <origin xyz="0 0 0" rpy="0 0 0"/>
+       <geometry>
+        <box size=".05 .05 .05"/>
+      </geometry>
+    </collision>
+</link>
+  <joint name="rgbd_joint" type="fixed">
+    <origin xyz="0.1 0 0.1" rpy="-1.5707 0  -1.5707" />
+    <parent link="chassis"/>
+    <child link="camera_rgbd"/>
+  </joint>
   <link name='hokuyo'>
     <pose>0 0 0.1 0 0 0</pose>
@@ -196,14 +224,3 @@
     <dynamics damping="1.0" friction="1.0"/>
   </joint>
-  <joint name="camera_optical_joint" type="fixed">
-    <origin xyz="0 0 0" rpy="-1.5707 0 -1.5707"/>
-    <parent link="camera"/>
-    <child link="camera_link_optical"/>
-  </joint>
-  <link name="camera_link_optical">
-  </link>
-<gazebo>
-  <plugin name="gazebo_ros_control" filename="libgazebo_ros_openni_kinect.so">
-  </plugin>
-</gazebo>
 </robot>
